Commit message: last version

File: uibk_robot_moveit_config/config/iis_robot_table.xacro (robot description, xacro)
@@ -35,5 +35,5 @@
 			      length="2.3"
 			      width="1.2"
-			      thickness="0.09">
+			      thickness="0.04">
     <!-- Place the table surface relative to the table plate -->
     <origin xyz="-0.4 -0.04 0" />
@@ -44,16 +44,16 @@
   </xacro:model_torso>
   <!-- left arm with gripper -->
-  <xacro:kuka_lwr_arm parent="world" name="left" right="-1">
+  <xacro:kuka_left_lwr_arm parent="world" name="left" right="-1">
     <origin xyz="-0.4923 0.7541 0.6295"
 	    rpy="1.9485 -0.2114 2.6898"/>
-  </xacro:kuka_lwr_arm>
+  </xacro:kuka_left_lwr_arm>
   <xacro:sdh_with_connector parent="left_arm_7_link" name="left_sdh">
     <origin rpy="0 0 ${-1/2 * M_PI}"/>
   </xacro:sdh_with_connector>
   <!-- right arm with gripper -->
-  <xacro:kuka_lwr_arm parent="world" name="right" right="1">
+  <xacro:kuka_right_lwr_arm parent="world" name="right" right="1">
     <origin xyz="-0.4962 0.5992 0.6335"
 	    rpy="-2.0628 0.7628 -3.1287"/>
-  </xacro:kuka_lwr_arm>
+  </xacro:kuka_right_lwr_arm>
   <xacro:sdh_with_connector parent="right_arm_7_link" name="right_sdh">
     <origin rpy="0 0 ${1/2 * M_PI}"/>
@@ -63,3 +63,18 @@
     <origin xyz="-0.4723 0.6767 0.85"/>
   </xacro:kit_head>
+  <!-- Kinect vision sensor -->
+  <!-- <link name="camera_link"/>
+  <joint name="kinect_visionSensor_joint" type="fixed" >
+	  <origin xyz="-0.40271 0.66297 0.796599"
+		  rpy="-1.69854 -0.0579848 -2.43762"/>
+	  <parent link="world_link" />
+	  <child link="camera_link" />
+  </joint> -->
+  <!-- simulator-->
+  <!-- <joint name="kinect_visionSensor_joint" type="fixed" >
+	  <origin xyz="-0.4568 0.6891 0.7516"
+		  rpy="2.2689 0.0 1.5708"/>
+	  <parent link="world_link" />
+	  <child link="kinect_visionSensor" />
+	</joint> -->
 </robot>

Commit message: switched back to old version

File: uibk_robot_moveit_config/config/iis_robot_table.xacro (robot description, xacro)
@@ -35,5 +35,5 @@
 			      length="2.3"
 			      width="1.2"
-			      thickness="0.04">
+			      thickness="0.09">
     <!-- Place the table surface relative to the table plate -->
     <origin xyz="-0.4 -0.04 0" />
@@ -44,16 +44,16 @@
   </xacro:model_torso>
   <!-- left arm with gripper -->
-  <xacro:kuka_left_lwr_arm parent="world" name="left" right="-1">
+  <xacro:kuka_lwr_arm parent="world" name="left" right="-1">
     <origin xyz="-0.4923 0.7541 0.6295"
 	    rpy="1.9485 -0.2114 2.6898"/>
-  </xacro:kuka_left_lwr_arm>
+  </xacro:kuka_lwr_arm>
   <xacro:sdh_with_connector parent="left_arm_7_link" name="left_sdh">
     <origin rpy="0 0 ${-1/2 * M_PI}"/>
   </xacro:sdh_with_connector>
   <!-- right arm with gripper -->
-  <xacro:kuka_right_lwr_arm parent="world" name="right" right="1">
+  <xacro:kuka_lwr_arm parent="world" name="right" right="1">
     <origin xyz="-0.4962 0.5992 0.6335"
 	    rpy="-2.0628 0.7628 -3.1287"/>
-  </xacro:kuka_right_lwr_arm>
+  </xacro:kuka_lwr_arm>
   <xacro:sdh_with_connector parent="right_arm_7_link" name="right_sdh">
     <origin rpy="0 0 ${1/2 * M_PI}"/>
@@ -63,18 +63,3 @@
     <origin xyz="-0.4723 0.6767 0.85"/>
   </xacro:kit_head>
-  <!-- Kinect vision sensor -->
-  <!-- <link name="camera_link"/>
-  <joint name="kinect_visionSensor_joint" type="fixed" >
-	  <origin xyz="-0.40271 0.66297 0.796599"
-		  rpy="-1.69854 -0.0579848 -2.43762"/>
-	  <parent link="world_link" />
-	  <child link="camera_link" />
-  </joint> -->
-  <!-- simulator-->
-  <!-- <joint name="kinect_visionSensor_joint" type="fixed" >
-	  <origin xyz="-0.4568 0.6891 0.7516"
-		  rpy="2.2689 0.0 1.5708"/>
-	  <parent link="world_link" />
-	  <child link="kinect_visionSensor" />
-	</joint> -->
 </robot>

Commit message: fixed robot model (removed collission in left arm origin state

File: uibk_robot_moveit_config/config/iis_robot_table.xacro (robot description, xacro)
@@ -33,9 +33,9 @@
   <xacro:model_table_surface name="table_surface"
 			      parent="table_plate"
-			      length="2.3"
+			      length="2.1"
 			      width="1.2"
 			      thickness="0.09">
     <!-- Place the table surface relative to the table plate -->
-    <origin xyz="-0.4 -0.04 0" />
+    <origin xyz="-0.4 -0.02 0" />
   </xacro:model_table_surface>
  <!-- add torso -->
